Commit message: update microwave

File: asset/partnet_mobility/7320/mobility.urdf (robot description, URDF)
Before this commit: robot partnet_c5d13a109a61060c178e7d331e641179, 3 links, 2 joints
Links:
- added link debug_red_dot; visual sphere radius=0.02
Joints:
- added joint debug_dot_joint: type fixed, parent link_1, child debug_red_dot, origin xyz=-0.7663123617888119 0.4711569999999998 0.39380938953471023
